File: hardware/ChromaSense_Breakout.kicad_sch (KiCad schematic)
At the start: 7 parts, among them J1 Grove, U1 TCS35303-2M, U2 AP2112K-1.8

Commit message: Schematic: fill title block (title, rev 1.1, date, author, licence)
Co-Authored-By: Claude Opus 5.5 <noreply@anthropic.com>
Claude-Session: https://claude.ai/code/session_01SnnjAyMwjQGxr5nzvAhxEy
Other:
- company: (none) -> OTH Regensburg
- title: (none) -> ChromaSense Breakout
Changed lines of the file:
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@@
 	(generator_version "10.0")
 	(paper "A4")
+	(title_block
+		(title "ChromaSense Breakout")
+		(date "17 April 2026")
+		(rev "1.1")
+		(company "OTH Regensburg")
+		(comment 1 "Vivek Wilson Neelamkavil")
+		(comment 2 "Licensed under CERN-OHL-P v2.")
+	)
 	(junction
 		(at 116.84 101.6)
